File: extras/schematics/pet_puller_shield/pet_puller_shield.kicad_pcb (KiCad board)
At the start: 2 copper layers, 1 part

Commit message: Update schematics
Parts:
- added C1: 220u, Capacitor_THT:CP_Radial_D8.0mm_P3.80mm, B.Cu at (166.4, 95.9)
- added D1: LED_Small, LED_THT:LED_D3.0mm, B.Cu at (174.5, 103.4)
- added J1: Jack-DC, Connector_BarrelJack:BarrelJack_GCT_DCJ200-10-A_Horizontal, B.Cu at (135.3, 104.8)
- added J2: Conn_01x02, Connector_JST:JST_EH_B2B-EH-A_1x02_P2.50mm_Vertical, B.Cu at (166.8, 103.3)
- added J3: Conn_01x02, Connector_JST:JST_EH_B2B-EH-A_1x02_P2.50mm_Vertical, B.Cu at (156.5, 104.3)
- added J4: Conn_01x02, Connector_JST:JST_NV_B02P-NV_1x02_P5.00mm_Vertical, B.Cu at (154.8, 95.8)
- added J5: Conn_01x04, Connector_JST:JST_EH_B4B-EH-A_1x04_P2.50mm_Vertical, B.Cu at (185.1, 101.5)
- added Q1: IRF540N, Package_TO_SOT_THT:TO-220-3_Vertical, B.Cu at (148.6, 124.2)
- added R1: 10k, Resistor_THT:R_Axial_DIN0204_L3.6mm_D1.6mm_P5.08mm_Horizontal, B.Cu at (174.5, 92.7)
- added R2: 220, Resistor_THT:R_Axial_DIN0204_L3.6mm_D1.6mm_P5.08mm_Horizontal, B.Cu at (164.0, 108.1)
- added R3: 10k, Resistor_THT:R_Axial_DIN0204_L3.6mm_D1.6mm_P5.08mm_Horizontal, B.Cu at (174.5, 95.8)
- added R4: 240, Resistor_THT:R_Axial_DIN0204_L3.6mm_D1.6mm_P5.08mm_Horizontal, B.Cu at (139.9, 115.3)
- added RV1: 1k, Potentiometer_THT:Potentiometer_Bourns_3339P_Vertical, B.Cu at (157.6, 114.6)
- added U1: LM317_TO-220, Package_TO_SOT_THT:TO-220-3_Vertical, B.Cu at (184.8, 91.0)
- added U2: MX1508_module, pet_puller:mx1508_module, B.Cu at (186.1, 101.1)
Connections:
- A1 pad 29: Net-(A1-Pad29) -> GND
- A1 pad 7: Net-(A1-Pad29) -> GND

Commit message: Updated schematics
Parts:
- added R5: 10k, Resistor_THT:R_Axial_DIN0204_L3.6mm_D1.6mm_P5.08mm_Horizontal, B.Cu at (137.2, 89.5)
- added R6: 220, Resistor_THT:R_Axial_DIN0204_L3.6mm_D1.6mm_P5.08mm_Horizontal, B.Cu at (137.0, 96.5)
- Q1, U1: footprint Package_TO_SOT_THT:TO-220-3_Vertical -> Package_TO_SOT_THT:TO-220-3_Horizontal_TabDown
- moved U1 58.8 mm to (135.6, 123.2), turned to 90 degrees
- moved D1 48.1 mm to (135.9, 132.1), turned to 0 degrees
- moved J4 31.8 mm to (186.1, 90.4), turned to -90 degrees
- moved J3 30.6 mm to (187.0, 102.3), turned to -90 degrees
- moved Q1 29.0 mm to (142.7, 95.8), turned to 90 degrees
- moved R2 29.0 mm to (146.1, 130.8)
- moved C1 27.6 mm to (140.3, 104.8), turned to 0 degrees
- moved J2 21.9 mm to (187.0, 111.8), turned to -90 degrees
- moved J5 19.2 mm to (185.1, 120.7), turned to -90 degrees
- moved R4 15.7 mm to (132.3, 129.0)
- moved U2 11.6 mm to (174.5, 99.8)
- moved RV1 9.53 mm to (152.7, 106.5), turned to 0 degrees
- moved R1 5.37 mm to (174.2, 98.0), turned to 0 degrees
- moved R3 3.92 mm to (174.0, 91.9), turned to 0 degrees
Connections:
- A1 pad 10: unconnected-(A1-Pad10) -> RUNOUT
- A1 pad 11: unconnected-(A1-Pad11) -> THERMISTOR
- A1 pad 17: M0 -> unconnected-(A1-Pad17)
- A1 pad 18: M1 -> unconnected-(A1-Pad18)
- A1 pad 19: M2 -> M0
- A1 pad 20: M3 -> M1
- A1 pad 21: HOTEND -> M2
- A1 pad 22: RUNOUT -> M3
- A1 pad 9: THERMISTOR -> HOTEND
- Q1 pad 1: HOTEND -> Net-(Q1-Pad1)
Routing:
- net +5V: track 0.00 -> 138.1 mm, vias 0 -> 2
- net +12V: track 0.00 -> 79.9 mm
- net +9V: track 0.00 -> 76.1 mm
- net Net-(J4-Pad1): track 0.00 -> 69.9 mm
- net HOTEND: track 0.00 -> 42.2 mm
- net Net-(J5-Pad4): track 0.00 -> 38.2 mm
- net Net-(J5-Pad3): track 0.00 -> 33.9 mm
- net THERMISTOR: track 0.00 -> 33.6 mm
- net Net-(R4-Pad1): track 0.00 -> 33.6 mm
- net RUNOUT: track 0.00 -> 31.0 mm, vias 0 -> 1
- net Net-(J5-Pad2): track 0.00 -> 27.3 mm
- net Net-(J5-Pad1): track 0.00 -> 22.7 mm
- net LED: track 0.00 -> 21.4 mm
- net M0: track 0.00 -> 13.8 mm
- net M1: track 0.00 -> 13.8 mm
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- added copper zone on B.Cu, net GND
- added copper zone on F.Cu, net GND
Other:
- board outline added: 75.4 x 53.8 mm

Commit message: Updated schematics
Routing:
- net Net-(J4-Pad1): track 69.9 -> 64.7 mm, vias 0 -> 1
- net +9V: track 76.1 -> 76.4 mm, vias 0 -> 1
Changed lines of the file:
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@@
   (segment (start 149.86 104.14) (end 142.875 111.125) (width 0.8) (layer "B.Cu") (net 5))
   (segment (start 182.245 104.14) (end 149.86 104.14) (width 0.8) (layer "B.Cu") (net 5))
+  (segment (start 182.88 92.71) (end 182.88 91.44) (width 1.6) (layer "F.Cu") (net 7))
+  (segment (start 182.88 91.44) (end 183.8875 90.4325) (width 1.6) (layer "F.Cu") (net 7))
+  (segment (start 183.8875 90.4325) (end 186.14 90.4325) (width 1.6) (layer "F.Cu") (net 7))
+  (via (at 182.88 92.71) (size 2) (drill 0.8) (layers "F.Cu" "B.Cu") (net 7))
   (segment (start 182.88 99.06) (end 179.705 102.235) (width 1.6) (layer "B.Cu") (net 7))
   (segment (start 139.7 93.98) (end 140.462 93.218) (width 1.6) (layer "B.Cu") (net 7))
   (segment (start 179.705 102.235) (end 147.32 102.235) (width 1.6) (layer "B.Cu") (net 7))
-  (segment (start 186.14 90.4325) (end 187.5875 90.4325) (width 1.6) (layer "B.Cu") (net 7))
   (segment (start 139.7 97.79) (end 139.7 93.98) (width 1.6) (layer "B.Cu") (net 7))
-  (segment (start 189.865 96.52) (end 187.325 99.06) (width 1.6) (layer "B.Cu") (net 7))
-  (segment (start 187.5875 90.4325) (end 189.865 92.71) (width 1.6) (layer "B.Cu") (net 7))
   (segment (start 140.462 93.218) (end 142.662 93.218) (width 1.6) (layer "B.Cu") (net 7))
-  (segment (start 189.865 92.71) (end 189.865 96.52) (width 1.6) (layer "B.Cu") (net 7))
-  (segment (start 187.325 99.06) (end 182.88 99.06) (width 1.6) (layer "B.Cu") (net 7))
   (segment (start 140.97 99.06) (end 139.7 97.79) (width 1.6) (layer "B.Cu") (net 7))
   (segment (start 144.145 99.06) (end 140.97 99.06) (width 1.6) (layer "B.Cu") (net 7))
   (segment (start 147.32 102.235) (end 144.145 99.06) (width 1.6) (layer "B.Cu") (net 7))
+  (segment (start 182.88 99.06) (end 182.88 92.71) (width 1.6) (layer "B.Cu") (net 7))
   (segment (start 169.164 95.25) (end 169.3465 95.4325) (width 0.25) (layer "F.Cu") (net 8))
   (segment (start 169.164 95.25) (end 168.91 94.996) (width 0.25) (layer "F.Cu") (net 8))
@@
   (segment (start 144.145 114.935) (end 144.235 114.935) (width 0.8) (layer "F.Cu") (net 28))
   (segment (start 150.114 109.056) (end 152.654 106.516) (width 0.8) (layer "F.Cu") (net 28))
+  (segment (start 178.435 127.381) (end 178.943 126.873) (width 0.8) (layer "F.Cu") (net 29))
+  (segment (start 178.435 128.27) (end 178.435 127.381) (width 0.8) (layer "F.Cu") (net 29))
   (segment (start 127.254 124.206) (end 130.81 120.65) (width 0.8) (layer "F.Cu") (net 29))
+  (segment (start 178.943 126.873) (end 178.943 124.5475) (width 0.8) (layer "F.Cu") (net 29))
   (segment (start 130.81 120.65) (end 135.55 120.65) (width 0.8) (layer "F.Cu") (net 29))
   (segment (start 127.254 129.032) (end 127.254 124.206) (width 0.8) (layer "F.Cu") (net 29))
-  (segment (start 178.943 127.127) (end 178.943 124.5475) (width 0.8) (layer "B.Cu") (net 29))
+  (via (at 178.435 128.27) (size 2) (drill 0.8) (layers "F.Cu" "B.Cu") (net 29))
   (segment (start 130.175 123.19) (end 135.255 128.27) (width 0.8) (layer "B.Cu") (net 29))
   (segment (start 130.81 120.65) (end 130.175 121.285) (width 0.8) (layer "B.Cu") (net 29))
   (segment (start 135.55 120.65) (end 130.81 120.65) (width 0.8) (layer "B.Cu") (net 29))
   (segment (start 130.175 121.285) (end 130.175 123.19) (width 0.8) (layer "B.Cu") (net 29))
-  (segment (start 177.8 128.27) (end 178.943 127.127) (width 0.8) (layer "B.Cu") (net 29))
+  (segment (start 177.8 128.27) (end 178.435 128.27) (width 0.8) (layer "B.Cu") (net 29))
   (segment (start 135.255 128.27) (end 177.8 128.27) (width 0.8) (layer "B.Cu") (net 29))
   (segment (start 138.405 132.08) (end 139.7 132.08) (width 0.8) (layer "F.Cu") (net 30))

Commit message: Updated schematics and gcode
Routing:
- net +5V: track 138.1 -> 137.6 mm
Changed lines of the file:
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@@
   (via (at 144.78 85.09) (size 2) (drill 0.8) (layers "F.Cu" "B.Cu") (net 5))
   (via (at 182.88 103.505) (size 2) (drill 0.8) (layers "F.Cu" "B.Cu") (net 5))
+  (segment (start 182.245 104.14) (end 149.86 104.14) (width 0.8) (layer "B.Cu") (net 5))
   (segment (start 142.875 86.995) (end 144.78 85.09) (width 0.8) (layer "B.Cu") (net 5))
   (segment (start 182.88 103.505) (end 182.245 104.14) (width 0.8) (layer "B.Cu") (net 5))
-  (segment (start 125.73 89.535) (end 128.27 86.995) (width 0.8) (layer "B.Cu") (net 5))
+  (segment (start 149.86 104.14) (end 143.51 110.49) (width 0.8) (layer "B.Cu") (net 5))
   (segment (start 125.73 107.95) (end 125.73 89.535) (width 0.8) (layer "B.Cu") (net 5))
   (segment (start 128.27 86.995) (end 142.875 86.995) (width 0.8) (layer "B.Cu") (net 5))
-  (segment (start 142.875 111.125) (end 128.905 111.125) (width 0.8) (layer "B.Cu") (net 5))
-  (segment (start 128.905 111.125) (end 125.73 107.95) (width 0.8) (layer "B.Cu") (net 5))
-  (segment (start 149.86 104.14) (end 142.875 111.125) (width 0.8) (layer "B.Cu") (net 5))
-  (segment (start 182.245 104.14) (end 149.86 104.14) (width 0.8) (layer "B.Cu") (net 5))
+  (segment (start 125.73 89.535) (end 128.27 86.995) (width 0.8) (layer "B.Cu") (net 5))
+  (segment (start 143.51 110.49) (end 128.27 110.49) (width 0.8) (layer "B.Cu") (net 5))
+  (segment (start 128.27 110.49) (end 125.73 107.95) (width 0.8) (layer "B.Cu") (net 5))
   (segment (start 182.88 92.71) (end 182.88 91.44) (width 1.6) (layer "F.Cu") (net 7))
   (segment (start 182.88 91.44) (end 183.8875 90.4325) (width 1.6) (layer "F.Cu") (net 7))

Commit message: Update schematics
Parts:
- added D2: 1N5402, Diode_THT:D_DO-201AD_P15.24mm_Horizontal, B.Cu at (141.6, 111.8)
- moved J1 1.67 mm to (135.3, 103.1)
- moved C1 0.38 mm to (140.3, 104.4)
Connections:
- J1 pad 3: GND -> (no net)
Routing:
- net +12V: track 79.9 -> 86.1 mm
- net +5V: track 137.6 -> 136.0 mm
Other:
- outline, holes or cut-outs redrawn

Commit message: Update schematics
Connections:
- A1 pad 10: RUNOUT -> unconnected-(A1-Pad10)
- A1 pad 17: unconnected-(A1-Pad17) -> RUNOUT
- J1 pad 3: (no net) -> GND
Routing:
- net RUNOUT: track 31.0 -> 42.6 mm, vias 1 -> 0
Changed lines of the file:
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@@
   (net 34 "Net-(J5-Pad4)")
   (net 35 "Net-(Q1-Pad1)")
-  (net 36 "unconnected-(A1-Pad17)")
+  (net 36 "unconnected-(A1-Pad10)")
   (net 37 "unconnected-(A1-Pad18)")
   (footprint "Module:Arduino_UNO_R2" (layer "F.Cu")
@@
       (net 19 "HOTEND") (pinfunction "A0") (pintype "bidirectional"))
     (pad "10" thru_hole oval (at 25.4 0 90) (size 1.6 1.6) (drill 1) (layers *.Cu *.Mask)
-      (net 20 "RUNOUT") (pinfunction "A1") (pintype "bidirectional"))
+      (net 36 "unconnected-(A1-Pad10)") (pinfunction "A1") (pintype "bidirectional+no_connect"))
     (pad "11" thru_hole oval (at 27.94 0 90) (size 1.6 1.6) (drill 1) (layers *.Cu *.Mask)
       (net 9 "THERMISTOR") (pinfunction "A2") (pintype "bidirectional"))
@@
       (net 14 "unconnected-(A1-Pad16)") (pinfunction "D1/TX") (pintype "bidirectional+no_connect"))
     (pad "17" thru_hole oval (at 30.48 48.26 90) (size 1.6 1.6) (drill 1) (layers *.Cu *.Mask)
-      (net 36 "unconnected-(A1-Pad17)") (pinfunction "D2") (pintype "bidirectional+no_connect"))
+      (net 20 "RUNOUT") (pinfunction "D2") (pintype "bidirectional"))
     (pad "18" thru_hole oval (at 27.94 48.26 90) (size 1.6 1.6) (drill 1) (layers *.Cu *.Mask)
       (net 37 "unconnected-(A1-Pad18)") (pinfunction "D3") (pintype "bidirectional+no_connect"))
@@
     (pad "2" thru_hole oval (at 0 -6.3 90) (size 4.2 2) (drill oval 3.2 1) (layers *.Cu *.Mask)
       (net 6 "GND") (pintype "passive"))
-    (pad "3" thru_hole oval (at 4.8 -2.9 90) (size 2 4.2) (drill oval 1 3.2) (layers *.Cu *.Mask))
+    (pad "3" thru_hole oval (at 4.8 -2.9 90) (size 2 4.2) (drill oval 1 3.2) (layers *.Cu *.Mask)
+      (net 6 "GND"))
     (model "${KICAD6_3DMODEL_DIR}/Connector_BarrelJack.3dshapes/BarrelJack_GCT_DCJ200-10-A_Horizontal.wrl"
       (offset (xyz 0 0 0))
@@
   (segment (start 143.51 83.185) (end 172.085 83.185) (width 0.8) (layer "F.Cu") (net 19))
   (segment (start 137.16 89.535) (end 143.51 83.185) (width 0.8) (layer "F.Cu") (net 19))
-  (segment (start 176.53 88.9) (end 176.53 85.09) (width 0.8) (layer "F.Cu") (net 20))
   (segment (start 187.025 111.78) (end 179.324 104.079) (width 0.8) (layer "F.Cu") (net 20))
   (segment (start 179.324 104.079) (end 179.324 98.044) (width 0.8) (layer "F.Cu") (net 20))
-  (via (at 176.53 88.9) (size 2) (drill 0.8) (layers "F.Cu" "B.Cu") (net 20))
-  (segment (start 179.324 98.044) (end 176.53 95.25) (width 0.8) (layer "B.Cu") (net 20))
-  (segment (start 176.53 95.25) (end 176.53 88.9) (width 0.8) (layer "B.Cu") (net 20))
+  (segment (start 181.61 114.046) (end 183.876 111.78) (width 0.8) (layer "B.Cu") (net 20))
+  (segment (start 183.876 111.78) (end 187.025 111.78) (width 0.8) (layer "B.Cu") (net 20))
+  (segment (start 181.61 133.35) (end 181.61 114.046) (width 0.8) (layer "B.Cu") (net 20))
   (segment (start 163.83 130.81) (end 145.415 130.81) (width 0.8) (layer "F.Cu") (net 21))
   (segment (start 164.85 133.35) (end 164.85 131.83) (width 0.8) (layer "F.Cu") (net 21))

Commit message: Update schematics
Routing:
- net RUNOUT: track 42.6 -> 42.9 mm, vias 0 -> 1
Changed lines of the file:
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@@
   (segment (start 143.51 83.185) (end 172.085 83.185) (width 0.8) (layer "F.Cu") (net 19))
   (segment (start 137.16 89.535) (end 143.51 83.185) (width 0.8) (layer "F.Cu") (net 19))
+  (segment (start 183.388 111.76) (end 187.005 111.76) (width 0.8) (layer "F.Cu") (net 20))
+  (segment (start 187.005 111.76) (end 187.025 111.78) (width 0.8) (layer "F.Cu") (net 20))
+  (segment (start 181.61 113.538) (end 183.388 111.76) (width 0.8) (layer "F.Cu") (net 20))
   (segment (start 187.025 111.78) (end 179.324 104.079) (width 0.8) (layer "F.Cu") (net 20))
   (segment (start 179.324 104.079) (end 179.324 98.044) (width 0.8) (layer "F.Cu") (net 20))
-  (segment (start 181.61 114.046) (end 183.876 111.78) (width 0.8) (layer "B.Cu") (net 20))
-  (segment (start 183.876 111.78) (end 187.025 111.78) (width 0.8) (layer "B.Cu") (net 20))
+  (via (at 181.61 113.538) (size 2) (drill 0.8) (layers "F.Cu" "B.Cu") (net 20))
   (segment (start 181.61 133.35) (end 181.61 114.046) (width 0.8) (layer "B.Cu") (net 20))
+  (segment (start 181.61 114.046) (end 181.61 113.538) (width 0.8) (layer "B.Cu") (net 20))
   (segment (start 163.83 130.81) (end 145.415 130.81) (width 0.8) (layer "F.Cu") (net 21))
   (segment (start 164.85 133.35) (end 164.85 131.83) (width 0.8) (layer "F.Cu") (net 21))

Commit message: Update schematics
Routing:
- net +5V: track 136.0 -> 69.0 mm
- net LED: track 21.4 -> 19.9 mm
- net HOTEND: track 42.2 -> 43.2 mm, vias 0 -> 1
- net M0: vias 0 -> 1
- net M1: vias 0 -> 1
- net M2: vias 0 -> 1
- net THERMISTOR: vias 0 -> 1
- net M3: vias 0 -> 1
- net +12V: vias 0 -> 1
