File: extras/schematics/pet_puller_shield/pet_puller_shield.kicad_pcb (KiCad board)
At the start: 2 copper layers, 75.4 x 53.8 mm, 19 parts, among them J1 Jack-DC, J2 Conn_01x02, J3 Conn_01x02, J4 Conn_01x02, J5 Conn_01x04, Q1 IRF540N, U1 LM317_TO-220, U2 MX1508_module

Commit message: Update schematics
Routing:
- net +5V: track 69.0 -> 83.1 mm, vias 2 -> 1
- net HOTEND: track 43.2 -> 42.3 mm
Changed lines of the file:
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@@
   (segment (start 187.025 114.28) (end 188.615 114.28) (width 0.8) (layer "F.Cu") (net 5))
   (segment (start 189.865 113.03) (end 189.865 107.595) (width 0.8) (layer "F.Cu") (net 5))
-  (segment (start 161.29 85.09) (end 164.592 88.392) (width 0.8) (layer "F.Cu") (net 5))
   (segment (start 187.025 104.755) (end 184.13 104.755) (width 0.8) (layer "F.Cu") (net 5))
   (segment (start 188.615 114.28) (end 189.865 113.03) (width 0.8) (layer "F.Cu") (net 5))
-  (segment (start 164.592 88.392) (end 175.006 88.392) (width 0.8) (layer "F.Cu") (net 5))
   (segment (start 184.13 104.755) (end 182.88 103.505) (width 0.8) (layer "F.Cu") (net 5))
   (via (at 182.88 103.505) (size 2) (drill 0.8) (layers "F.Cu" "B.Cu") (net 5))
-  (via (at 175.006 88.392) (size 2) (drill 0.8) (layers "F.Cu" "B.Cu") (net 5))
-  (segment (start 175.006 89.722478) (end 175.453522 90.17) (width 0.8) (layer "B.Cu") (net 5))
+  (segment (start 176.53 94.488) (end 176.53 90.17) (width 0.8) (layer "B.Cu") (net 5))
+  (segment (start 161.29 85.09) (end 163.068 83.312) (width 0.8) (layer "B.Cu") (net 5))
   (segment (start 187.452 99.568) (end 186.182 99.568) (width 0.8) (layer "B.Cu") (net 5))
   (segment (start 186.182 99.568) (end 182.88 102.87) (width 0.8) (layer "B.Cu") (net 5))
   (segment (start 183.388 87.63) (end 189.484 87.63) (width 0.8) (layer "B.Cu") (net 5))
   (segment (start 180.848 90.17) (end 183.388 87.63) (width 0.8) (layer "B.Cu") (net 5))
-  (segment (start 175.006 88.392) (end 175.006 89.722478) (width 0.8) (layer "B.Cu") (net 5))
+  (segment (start 176.53 90.17) (end 180.848 90.17) (width 0.8) (layer "B.Cu") (net 5))
+  (segment (start 170.688 83.312) (end 171.704 84.328) (width 0.8) (layer "B.Cu") (net 5))
   (segment (start 182.88 102.87) (end 182.88 103.505) (width 0.8) (layer "B.Cu") (net 5))
+  (segment (start 163.068 83.312) (end 170.688 83.312) (width 0.8) (layer "B.Cu") (net 5))
   (segment (start 189.484 87.63) (end 189.484 97.536) (width 0.8) (layer "B.Cu") (net 5))
+  (segment (start 171.704 95.504) (end 175.514 95.504) (width 0.8) (layer "B.Cu") (net 5))
   (segment (start 189.484 97.536) (end 187.452 99.568) (width 0.8) (layer "B.Cu") (net 5))
-  (segment (start 175.453522 90.17) (end 180.848 90.17) (width 0.8) (layer "B.Cu") (net 5))
+  (segment (start 171.704 84.328) (end 171.704 95.504) (width 0.8) (layer "B.Cu") (net 5))
+  (segment (start 175.514 95.504) (end 176.53 94.488) (width 0.8) (layer "B.Cu") (net 5))
   (segment (start 182.88 92.71) (end 182.88 91.44) (width 1.6) (layer "F.Cu") (net 7))
   (segment (start 182.88 91.44) (end 183.8875 90.4325) (width 1.6) (layer "F.Cu") (net 7))
@@
   (segment (start 168.91 133.35) (end 168.91 132.842) (width 0.8) (layer "B.Cu") (net 18))
   (segment (start 168.91 132.842) (end 167.386 131.318) (width 0.8) (layer "B.Cu") (net 18))
+  (segment (start 138.811 87.884) (end 137.16 89.535) (width 0.8) (layer "F.Cu") (net 19))
+  (segment (start 173.99 87.884) (end 138.811 87.884) (width 0.8) (layer "F.Cu") (net 19))
   (segment (start 136.995 91.44) (end 136.995 89.7) (width 0.8) (layer "F.Cu") (net 19))
   (segment (start 136.995 89.7) (end 137.16 89.535) (width 0.8) (layer "F.Cu") (net 19))
-  (segment (start 140.462 84.582) (end 140.462 86.233) (width 0.8) (layer "F.Cu") (net 19))
-  (segment (start 140.462 86.233) (end 137.16 89.535) (width 0.8) (layer "F.Cu") (net 19))
-  (via (at 140.462 84.582) (size 2) (drill 0.8) (layers "F.Cu" "B.Cu") (net 19))
-  (segment (start 173.99 85.09) (end 172.055 83.155) (width 0.8) (layer "B.Cu") (net 19))
-  (segment (start 172.055 83.155) (end 141.889 83.155) (width 0.8) (layer "B.Cu") (net 19))
-  (segment (start 141.889 83.155) (end 140.462 84.582) (width 0.8) (layer "B.Cu") (net 19))
+  (via (at 173.99 87.884) (size 2) (drill 0.8) (layers "F.Cu" "B.Cu") (net 19))
+  (segment (start 173.99 85.09) (end 173.99 87.884) (width 0.8) (layer "B.Cu") (net 19))
   (segment (start 183.388 111.76) (end 187.005 111.76) (width 0.8) (layer "F.Cu") (net 20))
   (segment (start 187.005 111.76) (end 187.025 111.78) (width 0.8) (layer "F.Cu") (net 20))
@@
     (polygon
       (pts
-        (xy 155.575 123.825)
-        (xy 149.225 123.825)
-        (xy 149.225 117.475)
-        (xy 155.575 117.475)
+        (xy 156.591 124.841)
+        (xy 148.082 124.841)
+        (xy 148.082 116.586)
+        (xy 156.591 116.586)
       )
     )
@@
     (polygon
       (pts
-        (xy 162.56 96.52)
-        (xy 156.21 96.52)
-        (xy 156.21 90.17)
-        (xy 162.56 90.17)
+        (xy 163.576 97.536)
+        (xy 155.194 97.536)
+        (xy 155.194 89.154)
+        (xy 163.576 89.154)
       )
     )
@@
       (pts
         (xy 145.544425 99.314)
-        (xy 166.626425 99.314)
-        (xy 166.626425 87.122)
-        (xy 145.544425 87.122)
+        (xy 166.880425 99.314)
+        (xy 166.880425 86.868)
+        (xy 145.544425 86.868)
       )
     )
@@
     (polygon
       (pts
-        (xy 138.176 126.746)
-        (xy 159.766 126.746)
-        (xy 159.766 114.554)
-        (xy 138.176 114.554)
-      )
-    )
+        (xy 137.668 127.254)
+        (xy 160.782 127.254)
+        (xy 160.782 114.3)
+        (xy 137.668 114.3)
+      )
+    )

Commit message: Update schematics
Parts:
- moved C1 0.10 mm to (140.4, 104.4)
Connections:
- A1 pad 18: unconnected-(A1-Pad18) -> HOTEND
- A1 pad 9: HOTEND -> unconnected-(A1-Pad9)
- J1 pad 3: GND -> (no net)
Routing:
- net HOTEND: track 42.3 -> 104.1 mm, vias 1 -> 0
Changed lines of the file:
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@@
   (net 35 "Net-(Q1-Pad1)")
   (net 36 "unconnected-(A1-Pad10)")
-  (net 37 "unconnected-(A1-Pad18)")
+  (net 37 "unconnected-(A1-Pad9)")
   (footprint "Module:Arduino_UNO_R2" (layer "F.Cu")
     (at 151.13 85.09)
@@
       (net 8 "+12V") (pinfunction "VIN") (pintype "power_in"))
     (pad "9" thru_hole oval (at 22.86 0 90) (size 1.6 1.6) (drill 1) (layers *.Cu *.Mask)
-      (net 19 "HOTEND") (pinfunction "A0") (pintype "bidirectional"))
+      (net 37 "unconnected-(A1-Pad9)") (pinfunction "A0") (pintype "bidirectional+no_connect"))
     (pad "10" thru_hole oval (at 25.4 0 90) (size 1.6 1.6) (drill 1) (layers *.Cu *.Mask)
       (net 36 "unconnected-(A1-Pad10)") (pinfunction "A1") (pintype "bidirectional+no_connect"))
@@
       (net 20 "RUNOUT") (pinfunction "D2") (pintype "bidirectional"))
     (pad "18" thru_hole oval (at 27.94 48.26 90) (size 1.6 1.6) (drill 1) (layers *.Cu *.Mask)
-      (net 37 "unconnected-(A1-Pad18)") (pinfunction "D3") (pintype "bidirectional+no_connect"))
+      (net 19 "HOTEND") (pinfunction "D3") (pintype "bidirectional"))
     (pad "19" thru_hole oval (at 25.4 48.26 90) (size 1.6 1.6) (drill 1) (layers *.Cu *.Mask)
       (net 15 "M0") (pinfunction "D4") (pintype "bidirectional"))
@@
   )
   (footprint "Capacitor_THT:CP_Radial_D8.0mm_P3.80mm" (layer "B.Cu")
-    (at 140.280698 104.394)
+    (at 140.378047 104.394)
     (descr "CP, Radial series, Radial, pin pitch=3.80mm, , diameter=8mm, Electrolytic Capacitor")
     (tags "CP Radial series Radial pin pitch 3.80mm  diameter 8mm Electrolytic Capacitor")
@@
     (property "Sheetname" "")
     (attr through_hole)
-    (fp_text reference "C1" (at 4.490906 7.239) (layer "B.SilkS")
+    (fp_text reference "C1" (at 5.671953 5.588) (layer "B.SilkS")
       (effects (font (size 1 1) (thickness 0.15)) (justify mirror))
     )
@@
     (pad "2" thru_hole oval (at 0 -6.3 90) (size 4.2 2) (drill oval 3.2 1) (layers *.Cu *.Mask)
       (net 6 "GND") (pintype "passive"))
-    (pad "3" thru_hole oval (at 4.8 -2.9 90) (size 2 4.2) (drill oval 1 3.2) (layers *.Cu *.Mask)
-      (net 6 "GND"))
+    (pad "3" thru_hole oval (at 4.8 -2.9 90) (size 2 4.2) (drill oval 1 3.2) (layers *.Cu *.Mask))
     (model "${KICAD6_3DMODEL_DIR}/Connector_BarrelJack.3dshapes/BarrelJack_GCT_DCJ200-10-A_Horizontal.wrl"
       (offset (xyz 0 0 0))
@@
   (segment (start 168.91 133.35) (end 168.91 132.842) (width 0.8) (layer "B.Cu") (net 18))
   (segment (start 168.91 132.842) (end 167.386 131.318) (width 0.8) (layer "B.Cu") (net 18))
-  (segment (start 138.811 87.884) (end 137.16 89.535) (width 0.8) (layer "F.Cu") (net 19))
-  (segment (start 173.99 87.884) (end 138.811 87.884) (width 0.8) (layer "F.Cu") (net 19))
   (segment (start 136.995 91.44) (end 136.995 89.7) (width 0.8) (layer "F.Cu") (net 19))
   (segment (start 136.995 89.7) (end 137.16 89.535) (width 0.8) (layer "F.Cu") (net 19))
-  (via (at 173.99 87.884) (size 2) (drill 0.8) (layers "F.Cu" "B.Cu") (net 19))
-  (segment (start 173.99 85.09) (end 173.99 87.884) (width 0.8) (layer "B.Cu") (net 19))
+  (segment (start 126.238 105.918) (end 128.016 107.696) (width 0.8) (layer "B.Cu") (net 19))
+  (segment (start 149.86 104.394) (end 170.577242 104.394) (width 0.8) (layer "B.Cu") (net 19))
+  (segment (start 146.558 107.696) (end 149.86 104.394) (width 0.8) (layer "B.Cu") (net 19))
+  (segment (start 170.577242 104.394) (end 179.07 112.886758) (width 0.8) (layer "B.Cu") (net 19))
+  (segment (start 180.61 131.81) (end 179.07 133.35) (width 0.8) (layer "B.Cu") (net 19))
+  (segment (start 180.61 119.396) (end 180.61 131.81) (width 0.8) (layer "B.Cu") (net 19))
+  (segment (start 126.238 97.028) (end 126.238 105.918) (width 0.8) (layer "B.Cu") (net 19))
+  (segment (start 179.07 112.886758) (end 179.07 117.856) (width 0.8) (layer "B.Cu") (net 19))
+  (segment (start 128.016 107.696) (end 146.558 107.696) (width 0.8) (layer "B.Cu") (net 19))
+  (segment (start 136.995 91.44) (end 131.826 91.44) (width 0.8) (layer "B.Cu") (net 19))
+  (segment (start 131.826 91.44) (end 126.238 97.028) (width 0.8) (layer "B.Cu") (net 19))
+  (segment (start 179.07 117.856) (end 180.61 119.396) (width 0.8) (layer "B.Cu") (net 19))
   (segment (start 183.388 111.76) (end 187.005 111.76) (width 0.8) (layer "F.Cu") (net 20))
   (segment (start 187.005 111.76) (end 187.025 111.78) (width 0.8) (layer "F.Cu") (net 20))
