File: extras/schematics/pet_puller_shield/pet_puller_shield.kicad_pcb (KiCad board)
At the start: 2 copper layers, 75.4 x 53.8 mm, 19 parts, among them J1 Jack-DC, J2 Conn_01x02, J3 Conn_01x02, J4 Conn_01x02, J5 Conn_01x04, Q1 IRF540N, U1 LM317_TO-220, U2 MX1508_module

Commit message: Update schematics
Parts:
- added J6: Conn_01x02, Connector_JST:JST_EH_B2B-EH-A_1x02_P2.50mm_Vertical, B.Cu at (128.3, 133.1)
- moved R4 0.76 mm to (132.3, 128.3)
Connections:
- J1 pad 3: (no net) -> GND
Routing:
- net +12V: track 86.1 -> 110.2 mm
- net Net-(R4-Pad1): track 33.6 -> 32.8 mm
- net +9V: track 76.4 -> 75.7 mm
Changed lines of the file:
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@@
   )
   (footprint "Resistor_THT:R_Axial_DIN0204_L3.6mm_D1.6mm_P5.08mm_Horizontal" (layer "B.Cu")
-    (at 132.334 129.032 180)
+    (at 132.334 128.27 180)
     (descr "Resistor, Axial_DIN0204 series, Axial, Horizontal, pin pitch=5.08mm, 0.167W, length*diameter=3.6*1.6mm^2, http://cdn-reichelt.de/documents/datenblatt/B400/1_4W%23YAG.pdf")
     (tags "Resistor Axial_DIN0204 series Axial Horizontal pin pitch 5.08mm 0.167W length 3.6mm diameter 1.6mm")
@@
       (net 19 "HOTEND") (pintype "passive"))
     (model "${KICAD6_3DMODEL_DIR}/Resistor_THT.3dshapes/R_Axial_DIN0204_L3.6mm_D1.6mm_P5.08mm_Horizontal.wrl"
+      (offset (xyz 0 0 0))
+      (scale (xyz 1 1 1))
+      (rotate (xyz 0 0 0))
+    )
+  )
+  (footprint "Connector_JST:JST_EH_B2B-EH-A_1x02_P2.50mm_Vertical" (layer "B.Cu")
+    (at 128.29 133.142)
+    (descr "JST EH series connector, B2B-EH-A (http://www.jst-mfg.com/product/pdf/eng/eEH.pdf), generated with kicad-footprint-generator")
+    (tags "connector JST EH vertical")
+    (property "Sheetfile" "pet_puller_shield.kicad_sch")
+    (property "Sheetname" "")
+    (attr through_hole)
+    (fp_text reference "J6" (at -3.83 0.208) (layer "B.SilkS")
+      (effects (font (size 1 1) (thickness 0.15)) (justify mirror))
+    )
+    (fp_text value "Conn_01x02" (at 1.25 -3.4) (layer "B.Fab")
+      (effects (font (size 1 1) (thickness 0.15)) (justify mirror))
+    )
+    (fp_text user "${REFERENCE}" (at 1.25 -1.5) (layer "B.Fab")
+      (effects (font (size 1 1) (thickness 0.15)) (justify mirror))
+    )
+    (fp_line (start -2.61 1.71) (end -2.61 -2.31) (layer "B.SilkS") (width 0.12))
+    (fp_line (start -2.91 -0.11) (end -2.91 -2.61) (layer "B.SilkS") (width 0.12))
+    (fp_line (start -2.61 -0.81) (end -1.61 -0.81) (layer "B.SilkS") (width 0.12))
+    (fp_line (start -2.11 1.21) (end 4.61 1.21) (layer "B.SilkS") (width 0.12))
+    (fp_line (start 4.11 -0.81) (end 4.11 -2.31) (layer "B.SilkS") (width 0.12))
+    (fp_line (start -2.61 0) (end -2.11 0) (layer "B.SilkS") (width 0.12))
+    (fp_line (start 4.61 1.21) (end 4.61 0) (layer "B.SilkS") (width 0.12))
+    (fp_line (start 4.61 0) (end 5.11 0) (layer "B.SilkS") (width 0.12))
+    (fp_line (start -2.91 -2.61) (end -0.41 -2.61) (layer "B.SilkS") (width 0.12))
+    (fp_line (start 5.11 1.71) (end -2.61 1.71) (layer "B.SilkS") (width 0.12))
+    (fp_line (start -2.61 -2.31) (end 5.11 -2.31) (layer "B.SilkS") (width 0.12))
+    (fp_line (start -1.61 -0.81) (end -1.61 -2.31) (layer "B.SilkS") (width 0.12))
+    (fp_line (start -2.11 0) (end -2.11 1.21) (layer "B.SilkS") (width 0.12))
+    (fp_line (start 5.11 -2.31) (end 5.11 1.71) (layer "B.SilkS") (width 0.12))
+    (fp_line (start 5.11 -0.81) (end 4.11 -0.81) (layer "B.SilkS") (width 0.12))
+    (fp_line (start -3 2.1) (end -3 -2.7) (layer "B.CrtYd") (width 0.05))
+    (fp_line (start 5.5 2.1) (end -3 2.1) (layer "B.CrtYd") (width 0.05))
+    (fp_line (start 5.5 -2.7) (end 5.5 2.1) (layer "B.CrtYd") (width 0.05))
+    (fp_line (start -3 -2.7) (end 5.5 -2.7) (layer "B.CrtYd") (width 0.05))
+    (fp_line (start 5 -2.2) (end 5 1.6) (layer "B.Fab") (width 0.1))
+    (fp_line (start -2.5 1.6) (end -2.5 -2.2) (layer "B.Fab") (width 0.1))
+    (fp_line (start 5 1.6) (end -2.5 1.6) (layer "B.Fab") (width 0.1))
+    (fp_line (start -2.5 -2.2) (end 5 -2.2) (layer "B.Fab") (width 0.1))
+    (fp_line (start -2.91 -0.11) (end -2.91 -2.61) (layer "B.Fab") (width 0.1))
+    (fp_line (start -2.91 -2.61) (end -0.41 -2.61) (layer "B.Fab") (width 0.1))
+    (pad "1" thru_hole roundrect (at 0 0) (size 1.7 2) (drill 1) (layers *.Cu *.Mask) (roundrect_rratio 0.147059)
+      (net 8 "+12V") (pinfunction "Pin_1") (pintype "passive"))
+    (pad "2" thru_hole oval (at 2.5 0) (size 1.7 2) (drill 1) (layers *.Cu *.Mask)
+      (net 6 "GND") (pinfunction "Pin_2") (pintype "passive"))
+    (model "${KICAD6_3DMODEL_DIR}/Connector_JST.3dshapes/JST_EH_B2B-EH-A_1x02_P2.50mm_Vertical.wrl"
       (offset (xyz 0 0 0))
       (scale (xyz 1 1 1))
@@
     (pad "2" thru_hole oval (at 0 -6.3 90) (size 4.2 2) (drill oval 3.2 1) (layers *.Cu *.Mask)
       (net 6 "GND") (pintype "passive"))
-    (pad "3" thru_hole oval (at 4.8 -2.9 90) (size 2 4.2) (drill oval 1 3.2) (layers *.Cu *.Mask))
+    (pad "3" thru_hole oval (at 4.8 -2.9 90) (size 2 4.2) (drill oval 1 3.2) (layers *.Cu *.Mask)
+      (net 6 "GND"))
     (model "${KICAD6_3DMODEL_DIR}/Connector_BarrelJack.3dshapes/BarrelJack_GCT_DCJ200-10-A_Horizontal.wrl"
       (offset (xyz 0 0 0))
@@
   (segment (start 182.88 99.06) (end 182.88 92.71) (width 1.6) (layer "B.Cu") (net 7))
   (segment (start 169.164 95.25) (end 169.3465 95.4325) (width 0.25) (layer "F.Cu") (net 8))
+  (segment (start 125.476 123.444) (end 130.81 118.11) (width 0.8) (layer "F.Cu") (net 8))
   (segment (start 140.280698 102.543302) (end 140.280698 104.394) (width 1.6) (layer "F.Cu") (net 8))
+  (segment (start 125.476 131.826) (end 125.476 123.444) (width 0.8) (layer "F.Cu") (net 8))
   (segment (start 135.55 118.11) (end 135.55 113.116) (width 1.6) (layer "F.Cu") (net 8))
   (segment (start 164.338 100.076) (end 169.164 95.25) (width 1.6) (layer "F.Cu") (net 8))
@@
   (segment (start 135.55 113.116) (end 136.906 111.76) (width 1.6) (layer "F.Cu") (net 8))
   (segment (start 138.684 104.394) (end 137.414 103.124) (width 1.6) (layer "F.Cu") (net 8))
+  (segment (start 126.792 133.142) (end 125.476 131.826) (width 0.8) (layer "F.Cu") (net 8))
   (segment (start 141.605 111.76) (end 141.605 109.093) (width 1.6) (layer "F.Cu") (net 8))
   (segment (start 141.605 109.093) (end 140.280698 107.768698) (width 1.6) (layer "F.Cu") (net 8))
+  (segment (start 130.81 118.11) (end 135.55 118.11) (width 0.8) (layer "F.Cu") (net 8))
   (segment (start 140.280698 104.394) (end 138.684 104.394) (width 1.6) (layer "F.Cu") (net 8))
   (segment (start 140.280698 107.768698) (end 140.280698 104.394) (width 1.6) (layer "F.Cu") (net 8))
   (segment (start 140.280698 102.543302) (end 142.748 100.076) (width 1.6) (layer "F.Cu") (net 8))
+  (segment (start 128.29 133.142) (end 126.792 133.142) (width 0.8) (layer "F.Cu") (net 8))
   (via (at 169.164 95.25) (size 2) (drill 0.8) (layers "F.Cu" "B.Cu") (net 8))
   (segment (start 168.91 85.09) (end 168.91 94.996) (width 1.6) (layer "B.Cu") (net 8))
@@
   (segment (start 144.235 114.935) (end 150.114 109.056) (width 0.8) (layer "F.Cu") (net 28))
   (segment (start 132.334 124.206) (end 133.35 123.19) (width 0.8) (layer "F.Cu") (net 28))
-  (segment (start 132.334 129.032) (end 132.334 124.206) (width 0.8) (layer "F.Cu") (net 28))
+  (segment (start 132.334 124.206) (end 132.334 128.27) (width 0.8) (layer "F.Cu") (net 28))
   (segment (start 135.55 123.19) (end 137.795 123.19) (width 0.8) (layer "F.Cu") (net 28))
   (segment (start 144.145 116.84) (end 144.145 114.935) (width 0.8) (layer "F.Cu") (net 28))
   (segment (start 144.145 114.935) (end 144.235 114.935) (width 0.8) (layer "F.Cu") (net 28))
   (segment (start 150.114 109.056) (end 152.654 106.516) (width 0.8) (layer "F.Cu") (net 28))
+  (segment (start 127.254 124.206) (end 127.254 128.27) (width 0.8) (layer "F.Cu") (net 29))
   (segment (start 178.435 127.381) (end 178.943 126.873) (width 0.8) (layer "F.Cu") (net 29))
   (segment (start 178.435 128.27) (end 178.435 127.381) (width 0.8) (layer "F.Cu") (net 29))
@@
   (segment (start 178.943 126.873) (end 178.943 124.5475) (width 0.8) (layer "F.Cu") (net 29))
   (segment (start 130.81 120.65) (end 135.55 120.65) (width 0.8) (layer "F.Cu") (net 29))
-  (segment (start 127.254 129.032) (end 127.254 124.206) (width 0.8) (layer "F.Cu") (net 29))
   (via (at 178.435 128.27) (size 2) (drill 0.8) (layers "F.Cu" "B.Cu") (net 29))
   (segment (start 130.175 123.19) (end 135.255 128.27) (width 0.8) (layer "B.Cu") (net 29))
