File: extras/schematics/pet_puller_shield/pet_puller_shield.kicad_sch (KiCad schematic)
At the start: 1 part

Commit message: Update schematics
Parts:
- added C1: 220u, Capacitor_THT:CP_Radial_D8.0mm_P3.80mm, symbol Device:C_Polarized
- added D1: LED_Small, LED_THT:LED_D3.0mm, symbol Device:LED_Small
- added J1: Jack-DC, Connector_BarrelJack:BarrelJack_GCT_DCJ200-10-A_Horizontal, symbol Connector:Jack-DC
- added J2, J3: Conn_01x02, Connector_JST:JST_EH_B2B-EH-A_1x02_P2.50mm_Vertical, symbol Connector_Generic:Conn_01x02
- added J4: Conn_01x02, Connector_JST:JST_NV_B02P-NV_1x02_P5.00mm_Vertical, symbol Connector_Generic:Conn_01x02
- added J5: Conn_01x04, Connector_JST:JST_EH_B4B-EH-A_1x04_P2.50mm_Vertical, symbol Connector_Generic:Conn_01x04
- added Q1: IRF540N, Package_TO_SOT_THT:TO-220-3_Vertical, symbol Transistor_FET:IRF540N
- added R1, R3: 10k, Resistor_THT:R_Axial_DIN0204_L3.6mm_D1.6mm_P5.08mm_Horizontal, symbol Device:R
- added R2: 220, Resistor_THT:R_Axial_DIN0204_L3.6mm_D1.6mm_P5.08mm_Horizontal, symbol Device:R
- added R4: 240, Resistor_THT:R_Axial_DIN0204_L3.6mm_D1.6mm_P5.08mm_Horizontal, symbol Device:R
- added RV1: 1k, Potentiometer_THT:Potentiometer_Bourns_3339P_Vertical, symbol Device:R_Potentiometer
- added U1: LM317_TO-220, Package_TO_SOT_THT:TO-220-3_Vertical, symbol Regulator_Linear:LM317_TO-220
- added U2: MX1508_module, pet_puller:mx1508_module, symbol pet_puller:MX1508_module
Connections:
- net +12V: now also C1.1, J1.1, J4.2 (Pin_2), U1.3 (VI)
- net +5V: now also J2.2 (Pin_2), J3.2 (Pin_2)
- net GND: now also A1.29 (GND), A1.7 (GND), C1.2, D1.1 (K), J1.2, Q1.3 (S), R1.1, R3.1, RV1.3, U2.2 (GND)
- net HOTEND: now also Q1.1 (G)
- net LED: now also R2.1
- net M0: now also U2.3 (IN1)
- net M1: now also U2.4 (IN2)
- net M2: now also U2.5 (IN3)
- net M3: now also U2.6 (IN4)
- net RUNOUT: now also J2.1 (Pin_1), R1.2
- net THERMISTOR: now also J3.1 (Pin_1), R3.2
- new net: R4.1, RV1.1, RV1.2, U1.1 (ADJ)
- new net: D1.2 (A), R2.2
- new net: J5.1 (Pin_1), U2.10 (OUT1)
- new net: J5.4 (Pin_4), U2.7 (OUT4)
- new net: J5.3 (Pin_3), U2.8 (OUT3)
- new net: J5.2 (Pin_2), U2.9 (OUT2)
- new net: J4.1 (Pin_1), Q1.2 (D)
- new net +9V: R4.2, U1.2 (VO), U2.1 (VCC)
Other:
- note added: "Arduino"
- note added: "Hotend control"
- note added: "Hotend temperature"
- note added: "LED indicator"
- note added: "Power input"
- note added: "Runout sensor"
- note added: "Stepper control"
- note added: "Stepper regulator"

Commit message: Updated schematics
Parts:
- added R5: 10k, Resistor_THT:R_Axial_DIN0204_L3.6mm_D1.6mm_P5.08mm_Horizontal, symbol Device:R
- added R6: 220, Resistor_THT:R_Axial_DIN0204_L3.6mm_D1.6mm_P5.08mm_Horizontal, symbol Device:R
- Q1, U1: footprint Package_TO_SOT_THT:TO-220-3_Vertical -> Package_TO_SOT_THT:TO-220-3_Horizontal_TabDown
Connections:
- net GND: now also R5.2
- net HOTEND: now also A1.9 (A0), R5.1, R6.2; no longer A1.21 (D6), Q1.1 (G)
- net M0: now also A1.19 (D4); no longer A1.17 (D2)
- net M1: now also A1.20 (D5); no longer A1.18 (D3)
- net M2: now also A1.21 (D6); no longer A1.19 (D4)
- net M3: now also A1.22 (D7); no longer A1.20 (D5)
- net RUNOUT: now also A1.10 (A1); no longer A1.22 (D7)
- net THERMISTOR: now also A1.11 (A2); no longer A1.9 (A0)
- new net: Q1.1 (G), R6.1

Commit message: Updated schematics and gcode
Other:
- moved on the sheet: C1
Changed lines of the file:
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@@
 (kicad_sch (version 20211123) (generator eeschema)
   (paper "A4")
+  (junction (at 52.07 26.67) (diameter 0) (color 0 0 0 0)
+  )
   (junction (at 86.36 31.75) (diameter 0) (color 0 0 0 0)
   )
@@
   (junction (at 81.28 69.85) (diameter 0) (color 0 0 0 0)
   )
-  (junction (at 46.99 34.29) (diameter 0) (color 0 0 0 0)
+  (junction (at 52.07 34.29) (diameter 0) (color 0 0 0 0)
   )
   (junction (at 173.99 31.75) (diameter 0) (color 0 0 0 0)
-  )
-  (junction (at 46.99 26.67) (diameter 0) (color 0 0 0 0)
   )
   (junction (at 88.9 60.96) (diameter 0) (color 0 0 0 0)
@@
     (stroke (width 0) (type default) (color 0 0 0 0))
   )
-  (wire (pts (xy 46.99 26.67) (xy 55.88 26.67))
+  (wire (pts (xy 41.91 26.67) (xy 52.07 26.67))
     (stroke (width 0) (type default) (color 0 0 0 0))
   )
@@
     (stroke (width 0) (type default) (color 0 0 0 0))
   )
+  (wire (pts (xy 52.07 26.67) (xy 55.88 26.67))
+    (stroke (width 0) (type default) (color 0 0 0 0))
+  )
   (polyline (pts (xy 147.32 45.72) (xy 147.32 16.51))
     (stroke (width 0) (type default) (color 0 0 0 0))
@@
     (stroke (width 0) (type default) (color 0 0 0 0))
   )
-  (wire (pts (xy 41.91 26.67) (xy 46.99 26.67))
-    (stroke (width 0) (type default) (color 0 0 0 0))
-  )
   (polyline (pts (xy 107.95 16.51) (xy 107.95 45.72))
     (stroke (width 0) (type default) (color 0 0 0 0))
@@
     (stroke (width 0) (type default) (color 0 0 0 0))
   )
-  (wire (pts (xy 41.91 34.29) (xy 46.99 34.29))
-    (stroke (width 0) (type default) (color 0 0 0 0))
-  )
   (wire (pts (xy 86.36 21.59) (xy 86.36 29.21))
     (stroke (width 0) (type default) (color 0 0 0 0))
@@
     (stroke (width 0) (type default) (color 0 0 0 0))
   )
+  (wire (pts (xy 52.07 34.29) (xy 55.88 34.29))
+    (stroke (width 0) (type default) (color 0 0 0 0))
+  )
   (wire (pts (xy 67.31 60.96) (xy 69.85 60.96))
     (stroke (width 0) (type default) (color 0 0 0 0))
@@
     (stroke (width 0) (type default) (color 0 0 0 0))
   )
-  (wire (pts (xy 46.99 34.29) (xy 55.88 34.29))
+  (wire (pts (xy 41.91 34.29) (xy 52.07 34.29))
     (stroke (width 0) (type default) (color 0 0 0 0))
   )
@@
     (pin "1")
   )
-  (symbol (lib_id "Device:C_Polarized") (at 46.99 30.48 0) (unit 1)
-    (in_bom yes) (on_board yes) (fields_autoplaced)
-    (property "Reference" "C1" (id 0) (at 49.911 28.7563 0)
+  (symbol (lib_id "Device:C_Polarized") (at 52.07 30.48 0) (unit 1)
+    (in_bom yes) (on_board yes) (fields_autoplaced)
+    (property "Reference" "C1" (id 0) (at 54.991 28.7563 0)
       (effects (font (size 1.27 1.27)) (justify left))
     )
-    (property "Value" "220u" (id 1) (at 49.911 31.2932 0)
+    (property "Value" "220u" (id 1) (at 54.991 31.2932 0)
       (effects (font (size 1.27 1.27)) (justify left))
     )
-    (property "Footprint" "Capacitor_THT:CP_Radial_D8.0mm_P3.80mm" (id 2) (at 47.9552 34.29 0)
-      (effects (font (size 1.27 1.27)) hide)
-    )
-    (property "Datasheet" "~" (id 3) (at 46.99 30.48 0)
-      (effects (font (size 1.27 1.27)) hide)
-    )
+    (property "Footprint" "Capacitor_THT:CP_Radial_D8.0mm_P3.80mm" (id 2) (at 53.0352 34.29 0)
+      (effects (font (size 1.27 1.27)) hide)
+    )
+    (property "Datasheet" "~" (id 3) (at 52.07 30.48 0)
+      (effects (font (size 1.27 1.27)) hide)
+    )

Commit message: Update schematics
Parts:
- added D2: 1N5402, Diode_THT:D_DO-201AD_P15.24mm_Horizontal, symbol Diode:1N5402
Connections:
- net +12V: now also D2.1 (K)
- net GND: now also D2.2 (A)
Changed lines of the file:
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@@
   (junction (at 86.36 31.75) (diameter 0) (color 0 0 0 0)
   )
-  (junction (at 41.91 34.29) (diameter 0) (color 0 0 0 0)
-  )
   (junction (at 77.47 69.85) (diameter 0) (color 0 0 0 0)
   )
+  (junction (at 36.83 33.02) (diameter 0) (color 0 0 0 0)
+  )
   (junction (at 81.28 69.85) (diameter 0) (color 0 0 0 0)
   )
@@
   (junction (at 240.03 80.01) (diameter 0) (color 0 0 0 0)
   )
-  (junction (at 41.91 26.67) (diameter 0) (color 0 0 0 0)
-  )
   (junction (at 53.34 67.31) (diameter 0) (color 0 0 0 0)
+  )
+  (junction (at 36.83 27.94) (diameter 0) (color 0 0 0 0)
+  )
+  (junction (at 45.72 34.29) (diameter 0) (color 0 0 0 0)
+  )
+  (junction (at 45.72 26.67) (diameter 0) (color 0 0 0 0)
   )
   (no_connect (at 252.73 39.37))
@@
     (stroke (width 0) (type default) (color 0 0 0 0))
   )
-  (wire (pts (xy 41.91 26.67) (xy 52.07 26.67))
+  (wire (pts (xy 39.37 26.67) (xy 45.72 26.67))
     (stroke (width 0) (type default) (color 0 0 0 0))
   )
@@
     (stroke (width 0) (type default) (color 0 0 0 0))
   )
+  (wire (pts (xy 45.72 26.67) (xy 52.07 26.67))
+    (stroke (width 0) (type default) (color 0 0 0 0))
+  )
   (polyline (pts (xy 21.59 49.53) (xy 21.59 86.36))
     (stroke (width 0) (type default) (color 0 0 0 0))
   )
+  (wire (pts (xy 36.83 24.13) (xy 36.83 27.94))
+    (stroke (width 0) (type default) (color 0 0 0 0))
+  )
   (wire (pts (xy 139.7 31.75) (xy 137.16 31.75))
     (stroke (width 0) (type default) (color 0 0 0 0))
@@
     (stroke (width 0) (type default) (color 0 0 0 0))
   )
+  (wire (pts (xy 45.72 34.29) (xy 52.07 34.29))
+    (stroke (width 0) (type default) (color 0 0 0 0))
+  )
   (polyline (pts (xy 63.5 49.53) (xy 63.5 86.36))
     (stroke (width 0) (type default) (color 0 0 0 0))
@@
     (stroke (width 0) (type default) (color 0 0 0 0))
   )
+  (wire (pts (xy 36.83 33.02) (xy 36.83 35.56))
+    (stroke (width 0) (type default) (color 0 0 0 0))
+  )
   (wire (pts (xy 242.57 80.01) (xy 242.57 77.47))
     (stroke (width 0) (type default) (color 0 0 0 0))
@@
     (stroke (width 0) (type default) (color 0 0 0 0))
   )
-  (wire (pts (xy 39.37 26.67) (xy 41.91 26.67))
-    (stroke (width 0) (type default) (color 0 0 0 0))
-  )
   (polyline (pts (xy 200.66 45.72) (xy 151.13 45.72))
     (stroke (width 0) (type default) (color 0 0 0 0))
@@
     (stroke (width 0) (type default) (color 0 0 0 0))
   )
-  (wire (pts (xy 39.37 34.29) (xy 41.91 34.29))
-    (stroke (width 0) (type default) (color 0 0 0 0))
-  )
   (wire (pts (xy 86.36 31.75) (xy 95.25 31.75))
     (stroke (width 0) (type default) (color 0 0 0 0))
@@
     (stroke (width 0) (type default) (color 0 0 0 0))
   )
-  (wire (pts (xy 41.91 34.29) (xy 52.07 34.29))
+  (wire (pts (xy 39.37 34.29) (xy 45.72 34.29))
     (stroke (width 0) (type default) (color 0 0 0 0))
   )
@@
     (pin "1")
   )
+  (symbol (lib_id "Diode:1N5402") (at 45.72 30.48 270) (unit 1)
+    (in_bom yes) (on_board yes)
+    (property "Reference" "D2" (id 0) (at 44.45 39.37 90)
+      (effects (font (size 1.27 1.27)) (justify left))
+    )
+    (property "Value" "1N5402" (id 1) (at 43.18 36.83 90)
+      (effects (font (size 1.27 1.27)) (justify left))
+    )
+    (property "Footprint" "Diode_THT:D_DO-201AD_P15.24mm_Horizontal" (id 2) (at 41.275 30.48 0)
+      (effects (font (size 1.27 1.27)) hide)
+    )
+    (property "Datasheet" "http://www.vishay.com/docs/88516/1n5400.pdf" (id 3) (at 45.72 30.48 0)
+      (effects (font (size 1.27 1.27)) hide)
+    )
+    (pin "1")
+    (pin "2")
+  )
   (symbol (lib_id "Device:C_Polarized") (at 52.07 30.48 0) (unit 1)
     (in_bom yes) (on_board yes) (fields_autoplaced)
@@
     (pin "1")
   )
-  (symbol (lib_id "power:PWR_FLAG") (at 41.91 34.29 180) (unit 1)
-    (in_bom yes) (on_board yes) (fields_autoplaced)
-    (property "Reference" "#FLG0102" (id 0) (at 41.91 36.195 0)
-      (effects (font (size 1.27 1.27)) hide)
-    )
-    (property "Value" "PWR_FLAG" (id 1) (at 41.91 38.7334 0))
-    (property "Footprint" "" (id 2) (at 41.91 34.29 0)
-      (effects (font (size 1.27 1.27)) hide)
-    )
-    (property "Datasheet" "~" (id 3) (at 41.91 34.29 0)
+  (symbol (lib_id "power:PWR_FLAG") (at 36.83 35.56 180) (unit 1)
+    (in_bom yes) (on_board yes) (fields_autoplaced)
+    (property "Reference" "#FLG0102" (id 0) (at 36.83 37.465 0)
+      (effects (font (size 1.27 1.27)) hide)
+    )
+    (property "Value" "PWR_FLAG" (id 1) (at 36.83 40.0034 0))
+    (property "Footprint" "" (id 2) (at 36.83 35.56 0)
+      (effects (font (size 1.27 1.27)) hide)
+    )
+    (property "Datasheet" "~" (id 3) (at 36.83 35.56 0)
       (effects (font (size 1.27 1.27)) hide)
     )
@@
     (pin "2")
   )
-  (symbol (lib_id "power:PWR_FLAG") (at 41.91 26.67 0) (unit 1)
-    (in_bom yes) (on_board yes) (fields_autoplaced)
-    (property "Reference" "#FLG0101" (id 0) (at 41.91 24.765 0)
-      (effects (font (size 1.27 1.27)) hide)
-    )
-    (property "Value" "PWR_FLAG" (id 1) (at 41.91 23.0942 0))
-    (property "Footprint" "" (id 2) (at 41.91 26.67 0)
-      (effects (font (size 1.27 1.27)) hide)
-    )
-    (property "Datasheet" "~" (id 3) (at 41.91 26.67 0)
+  (symbol (lib_id "power:PWR_FLAG") (at 36.83 24.13 0) (unit 1)
+    (in_bom yes) (on_board yes) (fields_autoplaced)
+    (property "Reference" "#FLG0101" (id 0) (at 36.83 22.225 0)
+      (effects (font (size 1.27 1.27)) hide)
+    )
+    (property "Value" "PWR_FLAG" (id 1) (at 36.83 20.5542 0))
+    (property "Footprint" "" (id 2) (at 36.83 24.13 0)
+      (effects (font (size 1.27 1.27)) hide)
+    )
+    (property "Datasheet" "~" (id 3) (at 36.83 24.13 0)
       (effects (font (size 1.27 1.27)) hide)
     )
@@
       (reference "D1") (unit 1) (value "LED_Small") (footprint "LED_THT:LED_D3.0mm")
     )
+    (path "/5ad7a0bb-d42f-4f0c-8236-96bc373b8ee1"
+      (reference "D2") (unit 1) (value "1N5402") (footprint "Diode_THT:D_DO-201AD_P15.24mm_Horizontal")
+    )
     (path "/3c5d0dfc-e6ad-419a-8ce4-3870822074e3"

Commit message: Update schematics
Connections:
- net RUNOUT: now also A1.17 (D2); no longer A1.10 (A1)
Changed lines of the file:
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@@
   (no_connect (at 252.73 39.37))
   (no_connect (at 252.73 44.45))
-  (no_connect (at 227.33 39.37))
   (no_connect (at 227.33 67.31))
   (no_connect (at 242.57 24.13))
+  (no_connect (at 252.73 52.07))
   (no_connect (at 252.73 59.69))
   (no_connect (at 227.33 59.69))
@@
     (effects (font (size 1.27 1.27)) (justify left bottom))
   )
-  (global_label "RUNOUT" (shape input) (at 252.73 52.07 0) (fields_autoplaced)
-    (effects (font (size 1.27 1.27)) (justify left))
-    (property "Intersheet References" "${INTERSHEET_REFS}" (id 0) (at 262.7026 52.1494 0)
-      (effects (font (size 1.27 1.27)) (justify left) hide)
-    )
-  )
   (global_label "M3" (shape output) (at 227.33 52.07 180) (fields_autoplaced)
     (effects (font (size 1.27 1.27)) (justify right))
@@
     )
   )
+  (global_label "RUNOUT" (shape input) (at 227.33 39.37 180) (fields_autoplaced)
+    (effects (font (size 1.27 1.27)) (justify right))
+    (property "Intersheet References" "${INTERSHEET_REFS}" (id 0) (at 217.3574 39.2906 0)
+      (effects (font (size 1.27 1.27)) (justify right) hide)
+    )
+  )

Commit message: Update schematics
Connections:
- net HOTEND: now also A1.18 (D3); no longer A1.9 (A0)
Changed lines of the file:
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@@
   (no_connect (at 252.73 44.45))
   (no_connect (at 227.33 67.31))
+  (no_connect (at 252.73 49.53))
   (no_connect (at 242.57 24.13))
   (no_connect (at 252.73 52.07))
@@
   (no_connect (at 227.33 62.23))
   (no_connect (at 252.73 62.23))
-  (no_connect (at 227.33 41.91))
   (wire (pts (xy 44.45 54.61) (xy 44.45 59.69))
     (stroke (width 0) (type default) (color 0 0 0 0))
@@
     )
   )
-  (global_label "HOTEND" (shape output) (at 252.73 49.53 0) (fields_autoplaced)
-    (effects (font (size 1.27 1.27)) (justify left))
-    (property "Intersheet References" "${INTERSHEET_REFS}" (id 0) (at 262.5212 49.6094 0)
-      (effects (font (size 1.27 1.27)) (justify left) hide)
-    )
-  )
+  (global_label "HOTEND" (shape output) (at 227.33 41.91 180) (fields_autoplaced)
+    (effects (font (size 1.27 1.27)) (justify right))
+    (property "Intersheet References" "${INTERSHEET_REFS}" (id 0) (at 217.5388 41.8306 0)
+      (effects (font (size 1.27 1.27)) (justify right) hide)
+    )
+  )
